Commit message: chore: adding changes

File: auv_d/urdf/auv_d.xacro (robot description, xacro)
@@ -9,5 +9,5 @@
 					1.0
 				</compensation>
-			</buoyancy>
+			</buoyancy>                z
         </link>
         <joint name="${name}" type="fixed">

File: v2_visual/urdf/auv_v2.xacro (robot description, xacro)
@@ -70,5 +70,5 @@
         <effort>40</effort>
         <name>m_star</name>
-        <map>>0 0 -1 0 0 0</map>
+        <map>0 0 -1 0 0 0</map>
       </thruster>
       <thruster>
@@ -244,5 +244,5 @@
   <!-- Sensor: Down Camera -->
   <link name="d_cam">
-    <collision>
+    <collision>1.5708
       <origin xyz="${cam_origin_offset}" rpy="0 0 0"/>
       <geometry>

File: v2_visual/urdf/task4_ball.xacro (robot description, xacro)
@@ -22,5 +22,5 @@
       <geometry>
         <mesh
-          filename="package://v2_visual/meshes/task4_ball_visual.STL" />
+          filename="package://v2_visual/meshes/belgian_gate.STL" />
       </geometry>
       <material
@@ -36,5 +36,5 @@
       <geometry>
         <mesh
-          filename="package://v2_visual/meshes/task4_ball_collision.STL" />
+          filename="package://v2_visual/meshes/belgian_gate.STL" />
       </geometry>
     </collision>
